File: PCB/Sazanami40.sch (KiCad schematic (older format))
At the start: 84 parts, among them SW1 SW_PUSH, SW10 SW_PUSH, SW11 SW_PUSH, SW12 SW_PUSH, SW13 SW_PUSH, SW14 SW_PUSH, SW15 SW_PUSH, SW16 SW_PUSH, SW17 SW_PUSH, SW18 SW_PUSH, SW19 SW_PUSH, SW2 SW_PUSH, SW20 SW_PUSH, SW21 SW_PUSH, SW22 SW_PUSH, SW23 SW_PUSH, SW24 SW_PUSH, SW25 SW_PUSH, SW26 SW_PUSH, SW27 SW_PUSH, SW28 SW_PUSH, SW29 SW_PUSH, SW3 SW_PUSH, SW30 SW_PUSH, SW31 SW_PUSH, SW32 SW_PUSH, SW33 SW_PUSH, SW34 SW_PUSH, SW35 SW_PUSH, SW36 SW_PUSH, SW37 SW_PUSH, SW38 SW_PUSH, SW39 SW_PUSH, SW4 SW_PUSH, SW40 SW_PUSH, SW41 SW_PUSH, SW42 SW_PUSH, SW43 SW_PUSH, SW5 SW_PUSH, SW6 SW_PUSH, SW7 SW_PUSH, SW8 SW_PUSH, SW9 SW_PUSH, U1 ProMicro

Commit message: layout complete :
Parts:
- added D13, D33: D, Diode_SMD:D_SOD-123, symbol Device:D
- added SW13, SW35: SW_PUSH, Keebio-Parts:MX_PCB_100H, symbol kbd:SW_PUSH
- SW1, SW10, SW11, SW12, SW2, SW3, SW4, SW5, SW6, SW7, SW8, SW9: footprint footprints:CHERRY_PCB_100H -> Keebio-Parts:MX_PCB_100H
- SW14: renamed from SW13; footprint footprints:CHERRY_PCB_100H -> Keebio-Parts:MX_PCB_100H
- SW15: renamed from SW14; footprint footprints:CHERRY_PCB_100H -> Keebio-Parts:MX_PCB_100H
- SW16: renamed from SW15; footprint footprints:CHERRY_PCB_100H -> Keebio-Parts:MX_PCB_100H
- SW17: renamed from SW16; footprint footprints:CHERRY_PCB_100H -> Keebio-Parts:MX_PCB_100H
- SW18: renamed from SW17; footprint footprints:CHERRY_PCB_100H -> Keebio-Parts:MX_PCB_100H
- SW19: renamed from SW18; footprint footprints:CHERRY_PCB_100H -> Keebio-Parts:MX_PCB_100H
- SW20: renamed from SW19; footprint footprints:CHERRY_PCB_100H -> Keebio-Parts:MX_PCB_100H
- SW21: renamed from SW20; footprint footprints:CHERRY_PCB_100H -> Keebio-Parts:MX_PCB_100H
- SW22: renamed from SW21; footprint footprints:CHERRY_PCB_100H -> Keebio-Parts:MX_PCB_100H
- SW23: renamed from SW22; footprint footprints:CHERRY_PCB_100H -> Keebio-Parts:MX_PCB_100H
- SW24: renamed from SW23; footprint footprints:CHERRY_PCB_100H -> Keebio-Parts:MX_PCB_100H
- SW25: renamed from SW24; footprint footprints:CHERRY_PCB_100H -> Keebio-Parts:MX_PCB_100H
- SW26: renamed from SW25; footprint footprints:CHERRY_PCB_100H -> Keebio-Parts:MX_PCB_100H
- SW27: renamed from SW26; footprint footprints:CHERRY_PCB_100H -> Keebio-Parts:MX_PCB_100H
- SW28: renamed from SW27; footprint footprints:CHERRY_PCB_100H -> Keebio-Parts:MX_PCB_100H
- SW29: renamed from SW28; footprint footprints:CHERRY_PCB_100H -> Keebio-Parts:MX_PCB_100H
- SW30: renamed from SW29; footprint footprints:CHERRY_PCB_100H -> Keebio-Parts:MX_PCB_100H
- SW31: renamed from SW30; footprint footprints:CHERRY_PCB_100H -> Keebio-Parts:MX_PCB_100H
- SW32: renamed from SW31; footprint footprints:CHERRY_PCB_100H -> Keebio-Parts:MX_PCB_100H
- SW33: renamed from SW32; footprint footprints:CHERRY_PCB_100H -> Keebio-Parts:MX_PCB_100H
- SW34: renamed from SW33; footprint footprints:CHERRY_PCB_100H -> Keebio-Parts:MX_PCB_100H
- SW36: renamed from SW34; footprint footprints:CHERRY_PCB_100H -> Keebio-Parts:MX_PCB_100H
- SW37: renamed from SW35; footprint footprints:CHERRY_PCB_100H -> Keebio-Parts:MX_PCB_100H
- SW38: renamed from SW36; footprint footprints:CHERRY_PCB_100H -> Keebio-Parts:MX_PCB_100H
- SW39: renamed from SW37; footprint footprints:CHERRY_PCB_100H -> Keebio-Parts:MX_PCB_100H
- SW40: renamed from SW38; footprint footprints:CHERRY_PCB_100H -> Keebio-Parts:MX_PCB_100H
- SW41: renamed from SW39; footprint footprints:CHERRY_PCB_100H -> Keebio-Parts:MX_PCB_100H
- SW42: renamed from SW40; footprint footprints:CHERRY_PCB_100H -> Keebio-Parts:MX_PCB_100H
- SW43: renamed from SW41; footprint footprints:CHERRY_PCB_100H -> Keebio-Parts:MX_PCB_100H
- SW44: renamed from SW42; footprint footprints:CHERRY_PCB_100H -> Keebio-Parts:MX_PCB_100H
- renumbered D13 to D14, D14 to D15, D15 to D16, D16 to D17, D17 to D18, D18 to D19, D19 to D20, D20 to D21, D21 to D22, D22 to D23, D23 to D24, D24 to D25, D25 to D26, D26 to D27, D27 to D28, D28 to D29, D29 to D30, D30 to D31, D31 to D32, D32 to D34, D33 to D35, D34 to D36, D35 to D37, D36 to D38, D37 to D39, D38 to D40, D39 to D41, D40 to D42, SW43 to SW45
Connections:
- net col3: now also SW13.1
- net col8: now also SW35.1
- net row2: now also D13.2 (A), D33.2 (A), SW13.2, SW35.2
- net row3: now also D13.1 (K), D33.1 (K)

Commit message: first draft PCB complete
Connections:
- net col0: now also U1.13 (B6)
- net col1: now also U1.14 (B2)
- net col10: now also U1.6 (SCL)
- net col11: now also U1.5 (SDA)
- net col2: now also U1.15 (B3)
- net col3: now also U1.16 (B1)
- net col4: now also U1.17 (F7)
- net col5: now also U1.18 (F6)
- net col6: now also U1.10 (E6)
- net col7: now also U1.9 (D7)
- net col8: now also U1.8 (C6)
- net col9: now also U1.7 (D4)
- net row0: now also U1.20 (F4)
- net row1: now also U1.19 (F5)
- net row2: now also U1.12 (B5); no longer D13.2 (A), D33.2 (A), SW13.2, SW35.2
- net row3: now also U1.11 (B4)
- net +5V renamed GND
- new net: D13.2 (A), SW13.2
- new net: D33.2 (A), SW35.2
- no-connect marks 0 -> 4
Changed lines of the file:
@@
 EESchema Schematic File Version 4
 LIBS:Sazanami40-cache
-EELAYER 29 0
+EELAYER 26 0
 EELAYER END
 $Descr A3 16535 11693
@@
 Wire Wire Line
 	14700 2000 15200 2000
-$Comp
-L keyboard_parts:GND #PWR05
-U 1 1 5CA439C8
-P 14950 2100
-F 0 "#PWR05" H 14950 2150 20  0001 C CNN
-F 1 "GND" H 14950 2159 30  0000 C CNN
-F 2 "" H 14950 2100 60  0000 C CNN
-F 3 "" H 14950 2100 60  0000 C CNN
-	1    14950 2100
-	1    0    0    -1
-$EndComp
-Wire Wire Line
-	14700 1800 14950 1800
-Wire Wire Line
-	14950 1800 14950 2100
 Text GLabel 14700 1900 2    50   Input ~ 0
 reset
-$Comp
-L keyboard_parts:GND #PWR01
-U 1 1 5CA43A18
-P 12900 2050
-F 0 "#PWR01" H 12900 2100 20  0001 C CNN
-F 1 "GND" H 12900 2109 30  0000 C CNN
-F 2 "" H 12900 2050 60  0000 C CNN
-F 3 "" H 12900 2050 60  0000 C CNN
-	1    12900 2050
-	1    0    0    -1
-$EndComp
 Wire Wire Line
 	13300 2000 12900 2000
@@
 F 3 "" H 14350 950 50  0001 C CNN
 	1    14350 950
-	1    0    0    -1
-$EndComp
-$Comp
-L keyboard_parts:GND #PWR02
-U 1 1 5CA43AF1
-P 13600 950
-F 0 "#PWR02" H 13600 1000 20  0001 C CNN
-F 1 "GND" H 13600 1009 30  0000 C CNN
-F 2 "" H 13600 950 60  0000 C CNN
-F 3 "" H 13600 950 60  0000 C CNN
-	1    13600 950
 	1    0    0    -1
 $EndComp
@@
 Text GLabel 13800 3500 0    50   Input ~ 0
 reset
-$Comp
-L keyboard_parts:GND #PWR04
-U 1 1 5CA43BF1
-P 14400 3500
-F 0 "#PWR04" H 14400 3550 20  0001 C CNN
-F 1 "GND" H 14400 3559 30  0000 C CNN
-F 2 "" H 14400 3500 60  0000 C CNN
-F 3 "" H 14400 3500 60  0000 C CNN
-	1    14400 3500
-	1    0    0    -1
-$EndComp
 $Comp
 L kbd:SW_PUSH SW1
@@
 $EndComp
 Wire Wire Line
-	5000 3600 5000 4100
-Connection ~ 5000 4100
-Wire Wire Line
 	4400 3300 4400 4100
 Connection ~ 4400 3300
@@
 $EndComp
 Wire Wire Line
-	9500 3600 9500 4100
-Connection ~ 9500 4100
-Wire Wire Line
 	8900 3300 8900 4100
 Connection ~ 8900 3300
@@
 	9500 4700 8600 4700
 Connection ~ 8600 4700
+$Comp
+L power:GND #PWR0101
+U 1 1 5CA60A81
+P 13600 950
+F 0 "#PWR0101" H 13600 700 50  0001 C CNN
+F 1 "GND" H 13605 777 50  0000 C CNN
+F 2 "" H 13600 950 50  0001 C CNN
+F 3 "" H 13600 950 50  0001 C CNN
+	1    13600 950
+	1    0    0    -1
+$EndComp
+Text GLabel 13300 2600 0    50   Input ~ 0
+col6
+Text GLabel 14700 2800 2    50   Input ~ 0
+col0
+Text GLabel 14700 2700 2    50   Input ~ 0
+col1
+Text GLabel 14700 2600 2    50   Input ~ 0
+col2
+Text GLabel 14700 2500 2    50   Input ~ 0
+col3
+Text GLabel 14700 2400 2    50   Input ~ 0
+col4
+Text GLabel 14700 2300 2    50   Input ~ 0
+col5
+Text GLabel 14700 2100 2    50   Input ~ 0
+row0
+Text GLabel 14700 2200 2    50   Input ~ 0
+row1
+Text GLabel 13300 2500 0    50   Input ~ 0
+col7
+Text GLabel 13300 2400 0    50   Input ~ 0
+col8
+Text GLabel 13300 2300 0    50   Input ~ 0
+col9
+Text GLabel 13300 2200 0    50   Input ~ 0
+col10
+Text GLabel 13300 2100 0    50   Input ~ 0
+col11
+Text GLabel 13300 2800 0    50   Input ~ 0
+row2
+Text GLabel 13300 2700 0    50   Input ~ 0
+row3
+NoConn ~ 14700 1700
+NoConn ~ 13300 1700
+NoConn ~ 13300 1800
+$Comp
+L power:GND #PWR0102
+U 1 1 5CA68914
+P 14400 3500
+F 0 "#PWR0102" H 14400 3250 50  0001 C CNN
+F 1 "GND" H 14405 3327 50  0000 C CNN
+F 2 "" H 14400 3500 50  0001 C CNN
+F 3 "" H 14400 3500 50  0001 C CNN
+	1    14400 3500
+	1    0    0    -1
+$EndComp
+$Comp
+L power:GND #PWR0103
+U 1 1 5CA68E60
+P 12900 2000
+F 0 "#PWR0103" H 12900 1750 50  0001 C CNN
+F 1 "GND" H 12905 1827 50  0000 C CNN
+F 2 "" H 12900 2000 50  0001 C CNN
+F 3 "" H 12900 2000 50  0001 C CNN
+	1    12900 2000
+	1    0    0    -1
+$EndComp
+$Comp
+L power:GND #PWR0104
+U 1 1 5CA6924D
+P 15100 2100
+F 0 "#PWR0104" H 15100 1850 50  0001 C CNN
+F 1 "GND" H 15105 1927 50  0000 C CNN
+F 2 "" H 15100 2100 50  0001 C CNN
+F 3 "" H 15100 2100 50  0001 C CNN
+	1    15100 2100
+	1    0    0    -1
+$EndComp
+Wire Wire Line
+	15100 1800 15100 2100
+Wire Wire Line
+	14700 1800 15100 1800
+NoConn ~ 5250 3250
 $EndSCHEMATC
